File: pcb/denmark.brd (EAGLE design)
At the start: 100 x 90 mm, 101 parts, among them IC1 74AHC1G32DBV, IC2 REG1117, U2 MB85RCSOIC8, X1 22-23-2021, X2 22-23-2031, X3 22-23-2051, X4 22-23-2021

Commit message: Cleanup Schematic
Parts:
- C12, C4: value 20n -> 20p
- Q1: value (none) -> 8.0 MHz
- R1, R2: value (none) -> 330
- R9: value NS -> 2.2k

Commit message: More BOM and schematic cleanup
Parts:
- renumbered U$1 to U1
